File: ORANGE_HAT/design/ORANGE_PI_4_PRO/ORANGE_PI_4_PRO.kicad_pcb (KiCad board)
At the start: 2 copper layers, 79 x 51 mm, 6 parts, among them P1 Conn_02x20_Odd_Even, P2 Conn_02x20_Odd_Even

Commit message: PWM code
Parts:
- added H1: MountingHole_2.1mm, MountingHole:MountingHole_2.1mm, F.Cu at (313.1, 31.5)
- added H1: MountingHole_2.1mm, MountingHole:MountingHole_2.1mm, F.Cu at (112.4, 94.3)
- added H1: MountingHole_2.1mm, MountingHole:MountingHole_2.1mm, F.Cu at (27.4, 25.9)
- added H1: MountingHole_2.1mm, MountingHole:MountingHole_2.1mm, F.Cu at (110.7, 170.1)
- added H1: MountingHole_2.1mm, MountingHole:MountingHole_2.1mm, F.Cu at (213.6, 28.0)
- added H1: MountingHole_2.1mm, MountingHole:MountingHole_2.1mm, F.Cu at (21.3, 165.8)
- added H1: MountingHole_2.1mm, MountingHole:MountingHole_2.1mm, F.Cu at (312.3, 103.8)
- added H1: MountingHole_2.1mm, MountingHole:MountingHole_2.1mm, F.Cu at (22.8, 96.4)
- added H1: MountingHole_2.1mm, MountingHole:MountingHole_2.1mm, F.Cu at (122.6, 27.6)
- added H1: MountingHole_2.1mm, MountingHole:MountingHole_2.1mm, F.Cu at (208.8, 174.6)
- added H2: MountingHole_2.2mm_M2, MountingHole:MountingHole_2.2mm_M2, F.Cu at (95.8, 96.4)
- added H2: MountingHole_2.2mm_M2, MountingHole:MountingHole_2.2mm_M2, F.Cu at (385.3, 103.8)
- added H2: MountingHole_2.2mm_M2, MountingHole:MountingHole_2.2mm_M2, F.Cu at (386.1, 31.5)
- added H2: MountingHole_2.2mm_M2, MountingHole:MountingHole_2.2mm_M2, F.Cu at (94.3, 165.8)
- added H2: MountingHole_2.2mm_M2, MountingHole:MountingHole_2.2mm_M2, F.Cu at (183.7, 170.1)
- added H2: MountingHole_2.2mm_M2, MountingHole:MountingHole_2.2mm_M2, F.Cu at (185.4, 94.3)
- added H2: MountingHole_2.2mm_M2, MountingHole:MountingHole_2.2mm_M2, F.Cu at (100.4, 25.9)
- added H2: MountingHole_2.2mm_M2, MountingHole:MountingHole_2.2mm_M2, F.Cu at (286.6, 28.0)
- added H2: MountingHole_2.2mm_M2, MountingHole:MountingHole_2.2mm_M2, F.Cu at (281.8, 174.6)
- added H2: MountingHole_2.2mm_M2, MountingHole:MountingHole_2.2mm_M2, F.Cu at (195.6, 27.6)
- added H3: MountingHole_2.1mm, MountingHole:MountingHole_2.1mm, F.Cu at (112.4, 139.3)
- added H3: MountingHole_2.1mm, MountingHole:MountingHole_2.1mm, F.Cu at (313.1, 76.5)
- added H3: MountingHole_2.1mm, MountingHole:MountingHole_2.1mm, F.Cu at (27.4, 70.9)
- added H3: MountingHole_2.1mm, MountingHole:MountingHole_2.1mm, F.Cu at (213.6, 73.0)
- added H3: MountingHole_2.1mm, MountingHole:MountingHole_2.1mm, F.Cu at (312.3, 148.8)
- added H3: MountingHole_2.1mm, MountingHole:MountingHole_2.1mm, F.Cu at (122.6, 72.7)
- added H3: MountingHole_2.1mm, MountingHole:MountingHole_2.1mm, F.Cu at (21.3, 210.8)
- added H3: MountingHole_2.1mm, MountingHole:MountingHole_2.1mm, F.Cu at (22.8, 141.4)
- added H3: MountingHole_2.1mm, MountingHole:MountingHole_2.1mm, F.Cu at (208.8, 219.6)
- added H3: MountingHole_2.1mm, MountingHole:MountingHole_2.1mm, F.Cu at (110.7, 215.1)
- added H4: MountingHole_2.1mm, MountingHole:MountingHole_2.1mm, F.Cu at (183.7, 215.1)
- added H4: MountingHole_2.1mm, MountingHole:MountingHole_2.1mm, F.Cu at (385.3, 148.8)
- added H4: MountingHole_2.1mm, MountingHole:MountingHole_2.1mm, F.Cu at (185.4, 139.3)
- added H4: MountingHole_2.1mm, MountingHole:MountingHole_2.1mm, F.Cu at (95.8, 141.4)
- added H4: MountingHole_2.1mm, MountingHole:MountingHole_2.1mm, F.Cu at (100.4, 70.9)
- added H4: MountingHole_2.1mm, MountingHole:MountingHole_2.1mm, F.Cu at (286.6, 73.0)
- added H4: MountingHole_2.1mm, MountingHole:MountingHole_2.1mm, F.Cu at (94.3, 210.8)
- added H4: MountingHole_2.1mm, MountingHole:MountingHole_2.1mm, F.Cu at (195.6, 72.7)
- added H4: MountingHole_2.1mm, MountingHole:MountingHole_2.1mm, F.Cu at (281.8, 219.6)
- added H4: MountingHole_2.1mm, MountingHole:MountingHole_2.1mm, F.Cu at (386.1, 76.5)
- added P1: Conn_02x20_Odd_Even, Connector_PinSocket_2.54mm:PinSocket_2x20_P2.54mm_Vertical, B.Cu at (39.3, 64.2)
- added P1: Conn_02x20_Odd_Even, Connector_PinSocket_2.54mm:PinSocket_2x20_P2.54mm_Vertical, B.Cu at (122.5, 208.3)
- added P1: Conn_02x20_Odd_Even, Connector_PinSocket_2.54mm:PinSocket_2x20_P2.54mm_Vertical, B.Cu at (220.7, 212.9)
- added P1: Conn_02x20_Odd_Even, Connector_PinSocket_2.54mm:PinSocket_2x20_P2.54mm_Vertical, B.Cu at (34.7, 134.7)
- added P1: Conn_02x20_Odd_Even, Connector_PinSocket_2.54mm:PinSocket_2x20_P2.54mm_Vertical, B.Cu at (33.2, 204.1)
- added P1: Conn_02x20_Odd_Even, Connector_PinSocket_2.54mm:PinSocket_2x20_P2.54mm_Vertical, B.Cu at (124.3, 132.6)
- added P1: Conn_02x20_Odd_Even, Connector_PinSocket_2.54mm:PinSocket_2x20_P2.54mm_Vertical, B.Cu at (324.2, 142.1)
- added P1: Conn_02x20_Odd_Even, Connector_PinSocket_2.54mm:PinSocket_2x20_P2.54mm_Vertical, B.Cu at (324.9, 69.8)
- added P1: Conn_02x20_Odd_Even, Connector_PinSocket_2.54mm:PinSocket_2x20_P2.54mm_Vertical, B.Cu at (134.5, 65.9)
- added P1: Conn_02x20_Odd_Even, Connector_PinSocket_2.54mm:PinSocket_2x20_P2.54mm_Vertical, B.Cu at (225.5, 66.3)
- added P2: Conn_02x20_Odd_Even, Connector_PinSocket_2.54mm:PinSocket_2x20_P2.54mm_Vertical, F.Cu at (134.5, 32.4)
- added P2: Conn_02x20_Odd_Even, Connector_PinSocket_2.54mm:PinSocket_2x20_P2.54mm_Vertical, F.Cu at (124.3, 99.0)
- added P2: Conn_02x20_Odd_Even, Connector_PinSocket_2.54mm:PinSocket_2x20_P2.54mm_Vertical, F.Cu at (122.5, 174.8)
- added P2: Conn_02x20_Odd_Even, Connector_PinSocket_2.54mm:PinSocket_2x20_P2.54mm_Vertical, F.Cu at (324.9, 36.3)
- added P2: Conn_02x20_Odd_Even, Connector_PinSocket_2.54mm:PinSocket_2x20_P2.54mm_Vertical, F.Cu at (39.3, 30.6)
- added P2: Conn_02x20_Odd_Even, Connector_PinSocket_2.54mm:PinSocket_2x20_P2.54mm_Vertical, F.Cu at (324.2, 108.6)
- added P2: Conn_02x20_Odd_Even, Connector_PinSocket_2.54mm:PinSocket_2x20_P2.54mm_Vertical, F.Cu at (220.7, 179.3)
- added P2: Conn_02x20_Odd_Even, Connector_PinSocket_2.54mm:PinSocket_2x20_P2.54mm_Vertical, F.Cu at (33.2, 170.6)
- added P2: Conn_02x20_Odd_Even, Connector_PinSocket_2.54mm:PinSocket_2x20_P2.54mm_Vertical, F.Cu at (34.7, 101.2)
- added P2: Conn_02x20_Odd_Even, Connector_PinSocket_2.54mm:PinSocket_2x20_P2.54mm_Vertical, F.Cu at (225.5, 32.7)
Routing:
- net GND: track 242.9 -> 2672.2 mm, vias 6 -> 66
- net /PL9: track 119.5 -> 1314.2 mm, vias 1 -> 11
- net +3.3V: track 118.7 -> 1305.8 mm, vias 3 -> 33
- net /PL12: track 107.1 -> 1177.6 mm, vias 1 -> 11
- net /PB5: track 101.4 -> 1115.7 mm, vias 3 -> 33
- net /PE2: track 95.7 -> 1052.8 mm, vias 3 -> 33
- net /PD1: track 90.3 -> 993.7 mm, vias 1 -> 11
- net /PD0: track 87.9 -> 967.3 mm, vias 1 -> 11
- net /PK24: track 83.6 -> 919.6 mm, vias 3 -> 33
- net /PD2: track 82.1 -> 903.4 mm, vias 1 -> 11
- net /PE1: track 80.9 -> 890.4 mm, vias 1 -> 11
- net /PL8: track 79.9 -> 878.4 mm, vias 1 -> 11
- net /PL4: track 76.6 -> 842.6 mm, vias 1 -> 11
- net /PD3: track 72.7 -> 800.1 mm, vias 1 -> 11
- net /PE3: track 72.5 -> 797.1 mm, vias 3 -> 33
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Other:
- board size 79 x 51 mm -> 370.8 x 199.7 mm
